File: HackPad/HackPad.kicad_pcb (KiCad board)
At the start: 2 copper layers, 100 x 100 mm, 39 parts, among them J1 Conn_01x14, J2 Conn_01x14, SW1 SW_Push, SW10 SW_Push, SW11 SW_Push, SW12 SW_Push, SW13 SW_Push, SW2 SW_Push, SW3 SW_Push, SW4 SW_Push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

Commit message: gerber
Parts:
- added BP1: Break Off, Mousebites:mouse-bite-2mm-slot, F.Cu at (106.2, 90.8)
- added BP2: Break Off, Mousebites:mouse-bite-2mm-slot, F.Cu at (193.2, 90.8)
- added BP3: Break Off, Mousebites:mouse-bite-2mm-slot, F.Cu at (151.0, 90.8)
- moved H7 2.48 mm to (195.0, 124.0)
- moved H6 0.57 mm to (193.5, 98.5)
Other:
- outline, holes or cut-outs redrawn
