File: HackPad/HackPad.kicad_sch (KiCad schematic)
At the start: 39 parts, among them J1 Conn_01x14, J2 Conn_01x14, SW1 SW_Push, SW10 SW_Push, SW11 SW_Push, SW12 SW_Push, SW13 SW_Push, SW2 SW_Push, SW3 SW_Push, SW4 SW_Push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

Commit message: gerber
Parts:
- added BP1, BP2, BP3: Break Off, Mousebites:mouse-bite-2mm-slot, symbol Mechanical:MountingHole
Other:
- moved on the sheet: J1, J2
